File: 8042board.sch (KiCad schematic (older format))
At the start: 17 parts, among them J1 To TM1637 display, SW1 Hour, SW2 Min, U1 8042, U2 2764, Y1 6/12MHz

Commit message: Update design files, provide Gerber fab files
Parts:
- removed U2: 2764, Package_DIP:DIP-28_W15.24mm, symbol Memory_EPROM:2764
- added C6: 10uF, Capacitor_THT:CP_Radial_D5.0mm_P2.50mm, symbol Device:CP_Small
- added H1, H2: MountingHole, MountingHole:MountingHole_3.5mm, symbol Mechanical:MountingHole
- added J2: Power, Connector_PinHeader_2.54mm:PinHeader_1x02_P2.54mm_Vertical, symbol Connector_Generic:Conn_01x02
- added JP2: LED, Connector_PinHeader_2.54mm:PinHeader_1x02_P2.54mm_Vertical, symbol Device:Jumper_NO_Small
- added U2: 27128, Package_DIP:DIP-28_W15.24mm_Socket, symbol Memory_EPROM:27128
- C1: value 1µF -> 1uF; footprint (none) -> Capacitor_THT:CP_Radial_D5.0mm_P2.50mm
- C2, C3: footprint (none) -> Capacitor_THT:C_Disc_D3.0mm_W1.6mm_P2.50mm
- C4, C5: value 0.1µF -> 0.1uF; footprint (none) -> Capacitor_THT:C_Rect_L7.0mm_W2.5mm_P5.00mm
- D1: footprint (none) -> LED_THT:LED_D5.0mm
- D2: footprint (none) -> Diode_THT:D_A-405_P7.62mm_Horizontal
- J1: footprint (none) -> Connector_PinHeader_2.54mm:PinHeader_1x07_P2.54mm_Vertical; symbol Connector_Generic:Conn_01x02 -> Connector_Generic:Conn_01x07
- JP1: footprint (none) -> Connector_PinHeader_2.54mm:PinHeader_1x03_P2.54mm_Vertical
- R1: value 1kΩ -> 1k; footprint (none) -> Resistor_THT:R_Axial_DIN0207_L6.3mm_D2.5mm_P10.16mm_Horizontal
- R2, R3: value 22kΩ -> 22k; footprint (none) -> Resistor_THT:R_Axial_DIN0207_L6.3mm_D2.5mm_P10.16mm_Horizontal
- SW1, SW2: footprint (none) -> Button_Switch_THT:SW_PUSH_6mm_H4.3mm
- U1: footprint (none) -> Package_DIP:DIP-40_W15.24mm_Socket
- Y1: footprint (none) -> Crystal:Crystal_HC18-U_Vertical
Connections:
- net +5V: now also J1.6 (Pin_6), C6.1, J2.1 (Pin_1), JP2.1, U2.1 (VPP), U2.27 (~PGM), U2.28 (VCC); no longer R1.1
- net A0: now also U2.10 (A0)
- net A1: now also U2.9 (A1)
- net A10: now also U2.21 (A10)
- net A2: now also U2.8 (A2)
- net A3: now also U2.7 (A3)
- net A4: now also U2.6 (A4)
- net A5: now also U2.5 (A5)
- net A6: now also U2.4 (A6)
- net A7: now also U2.3 (A7)
- net A8: now also U2.25 (A8)
- net A9: now also U2.24 (A9)
- net D0: now also U2.11 (D0)
- net D1: now also U2.12 (D1)
- net D2: now also U2.13 (D2)
- net D3: now also U2.15 (D3)
- net D4: now also U2.16 (D4)
- net D5: now also U2.17 (D5)
- net D6: now also U2.18 (D6)
- net D7: now also U2.19 (D7)
- net GND: now also J1.7 (Pin_7), C6.2, J2.2 (Pin_2), U2.14 (GND), U2.2 (A12), U2.22 (~OE), U2.23 (A11), U2.26 (A13)
- net at U1.11 (SYNC): now also U2.20 (~CE)
- net at U1.24 (P2.3): now also J1.1 (Pin_1)
- net at U1.35 (P2.4): now also J1.2 (Pin_2)
- net at D1.1 (K), U1.36 (P2.5): now also J1.3 (Pin_3)
- net at U1.37 (P2.6): now also J1.4 (Pin_4); no longer J1.1 (Pin_1)
- net at U1.38 (P2.7): now also J1.5 (Pin_5); no longer J1.2 (Pin_2)
- new net: JP2.2, R1.1
- no-connect marks 2 -> 0
Other:
- note added: "+5V"
- note added: "GND"
- note removed: "2018-10-28"
- note removed: "8042 board"
- moved on the sheet: C1, C2, C3, C4, C5, D1, D2, JP1, R1, R2, R3, SW1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
